Commit message: ugv are expressed in xacro

File: models/ground_stations/urdf/ground_station_0.urdf (robot description, URDF)
Before this commit: robot base_station_3, 1 links, 0 joints
Links:
- removed link base_station_link
- added link ground_station_link, mass 1.0; collision cylinder length=1.0 radius=0.5; visual cylinder length=1.0 radius=0.5

File: models/ground_stations/urdf/ground_station_1.urdf (robot description, URDF)
Before this commit: robot base_station_4, 1 links, 0 joints
Links:
- removed link base_station_link
- added link ground_station_link, mass 1.0; collision cylinder length=1.0 radius=0.5; visual cylinder length=1.0 radius=0.5

File: models/ground_stations/urdf/ground_station_2.urdf (robot description, URDF)
Before this commit: robot base_station_1, 1 links, 0 joints
Links:
- removed link base_station_link
- added link ground_station_link, mass 1.0; collision cylinder length=1.0 radius=0.5; visual cylinder length=1.0 radius=0.5

File: models/ground_stations/urdf/ground_station_3.urdf (robot description, URDF)
Before this commit: robot base_station_0, 1 links, 0 joints
Links:
- removed link base_station_link
- added link ground_station_link, mass 1.0; collision cylinder length=1.0 radius=0.5; visual cylinder length=1.0 radius=0.5

File: models/ground_stations/urdf/ground_station_4.urdf (robot description, URDF)
Before this commit: robot base_station_2, 1 links, 0 joints
Links:
- removed link base_station_link
- added link ground_station_link, mass 1.0; collision cylinder length=1.0 radius=0.5; visual cylinder length=1.0 radius=0.5

File: models/xacro_base/ground_station.xacro (robot description, xacro)
@@ -6,5 +6,5 @@
     </material>
     <xacro:insert_block name="origin" />
-    <link name="base_station_link">
+    <link name="ground_station_link">
       <inertial>
         <mass value="1.0" />
@@ -18,5 +18,5 @@
         />
       </inertial>
-      <visual name="base_station_visual">
+      <visual name="ground_station_visual">
         <geometry>
           <cylinder radius="0.5" length="1.0"/>
@@ -24,5 +24,5 @@
         <material name="red"/>
       </visual>
-      <collision name="base_station_collision">
+      <collision name="ground_station_collision">
         <geometry>
           <cylinder radius="0.5" length="1.0"/>
