Commit message: bug fix -antennaRotation

File: models/ground_stations/xacro/ground_station_0.xacro (robot description, xacro)
@@ -3,5 +3,5 @@
   <xacro:include filename="/home/haruki/Desktop/ugv_comms_in_gazebo/models/xacro_base/ground_station.xacro" />
   <xacro:base_staion>
-    <origin xyz="10 3 0.5" rpy="0 0 0" />
+    <origin xyz="5 3 0.5" rpy="0 0 0" />
     <address>ground_station_0</address>
     <topic>ground_station_0/rx</topic>

File: models/multicopters/urdf/multicopter_0.urdf (robot description, URDF)
Before this commit: robot multicopter_0, 5 links, 4 joints
Joints:
- joint multicopter_0/rotor_0_joint: origin xyz=0.13 -0.22 0.023 rpy=0 -0 0 -> xyz=0.13 -0.22 0.023 rpy=0 0 0
- joint multicopter_0/rotor_1_joint: origin xyz=-0.13 0.2 0.023 rpy=0 -0 0 -> xyz=-0.13 0.2 0.023 rpy=0 0 0
- joint multicopter_0/rotor_2_joint: origin xyz=0.13 0.22 0.023 rpy=0 -0 0 -> xyz=0.13 0.22 0.023 rpy=0 0 0
- joint multicopter_0/rotor_3_joint: origin xyz=-0.13 -0.2 0.023 rpy=0 -0 0 -> xyz=-0.13 -0.2 0.023 rpy=0 0 0

File: models/multicopters/xacro/multicopter_0.xacro (robot description, xacro)
@@ -4,12 +4,12 @@
   <xacro:include filename="/home/haruki/Desktop/ugv_comms_in_gazebo/models/xacro_base/multicopter.xacro" />
   <!-- <origin xyz="0.0 0.0 0.053302" rpy="0 0 0" /> -->
-  <origin xyz="0.0 0.0 1.0" rpy="0 0 0" />
+  <origin xyz="0.0 0.0 2.0" rpy="0 0 0" />
   <!-- frame -->
   <xacro:base name="${entity_name}"/>
   <!-- rotor -->
-  <xacro:rotor name="${entity_name}" num="0" rel_pos="0.13 -0.22 0.023" rel_rot="0 -0 0"/>
-  <xacro:rotor name="${entity_name}" num="1" rel_pos="-0.13 0.2 0.023" rel_rot="0 -0 0"/>
-  <xacro:rotor name="${entity_name}" num="2" rel_pos="0.13 0.22 0.023" rel_rot="0 -0 0"/>
-  <xacro:rotor name="${entity_name}" num="3" rel_pos="-0.13 -0.2 0.023" rel_rot="0 -0 0"/>
+  <xacro:rotor name="${entity_name}" num="0" rel_pos="0.13 -0.22 0.023" rel_rot="0 0 0"/>
+  <xacro:rotor name="${entity_name}" num="1" rel_pos="-0.13 0.2 0.023" rel_rot="0 0 0"/>
+  <xacro:rotor name="${entity_name}" num="2" rel_pos="0.13 0.22 0.023" rel_rot="0 0 0"/>
+  <xacro:rotor name="${entity_name}" num="3" rel_pos="-0.13 -0.2 0.023" rel_rot="0 0 0"/>
   <!-- gazebo  -->
   <xacro:gazebo name="${entity_name}"/>

File: models/ugvs/xacro/ugv_0.xacro (robot description, xacro)
@@ -3,5 +3,5 @@
   <xacro:include filename="/home/haruki/Desktop/ugv_comms_in_gazebo/models/xacro_base/ugv.xacro" />
   <!-- pose -->
-  <origin xyz="-2.0 0.0 0.5" rpy="0 0 0" />
+  <origin xyz="2.0 0.0 0.5" rpy="0 0 0" />
   <!-- chassis -->
   <xacro:chassis mass="10.0" width="2.0" height="1.0" dimension="0.5" material="blue"/>
