Commit message: function which is able to switch srcNode is made(ver.1)

File: models/ground_stations/xacro/ground_station_1.xacro (robot description, xacro)
@@ -3,5 +3,5 @@
   <xacro:include filename="/home/haruki/Desktop/ugv_comms_in_gazebo/models/xacro_base/ground_station.xacro" />
   <xacro:base_staion>
-    <origin xyz="15 3 0.5" rpy="0 0 0" />
+    <origin xyz="7.5 3 0.5" rpy="0 0 0" />
     <address>ground_station_1</address>
     <topic>ground_station_1/rx</topic>

File: models/ground_stations/xacro/ground_station_2.xacro (robot description, xacro)
@@ -3,5 +3,5 @@
   <xacro:include filename="/home/haruki/Desktop/ugv_comms_in_gazebo/models/xacro_base/ground_station.xacro" />
   <xacro:base_staion>
-    <origin xyz="20 3 0.5" rpy="0 0 0" />
+    <origin xyz="10 3 0.5" rpy="0 0 0" />
     <address>ground_station_2</address>
     <topic>ground_station_2/rx</topic>
