Commit message: adapt relative path

File: models/ground_station_antennas/xacro/ground_station_antenna_0.xacro (robot description, xacro)
@@ -1,8 +1,9 @@
 <?xml version="1.0"?>
 <robot name="ground_station_antenna_0" xmlns:xacro="http://ros.org/wiki/xacro">
+  <xacro:arg name="current_dirpath" default=""/>
   <xacro:property name="entity_name" value="ground_station_antenna_0"/>
-  <xacro:property name="pos_2d" value="5 3"/>
+  <xacro:property name="pos_2d" value="10 3"/>
   <xacro:property name="antenna_height" value="1.8"/>
-  <xacro:include filename="/home/haruki/Desktop/ugv_comms_in_gazebo/models/xacro_base/ground_station_antenna.xacro" />
+  <xacro:include filename="$(arg current_dirpath)/models/xacro_base/ground_station_antenna.xacro" />
   <origin xyz="${pos_2d} ${antenna_height}" rpy="0 0 0"/>
   <xacro:ground_station_antenna name="${entity_name}" antenna_height="${antenna_height}"/>

File: models/ground_station_antennas/xacro/ground_station_antenna_1.xacro (robot description, xacro)
@@ -1,8 +1,9 @@
 <?xml version="1.0"?>
 <robot name="ground_station_antenna_1" xmlns:xacro="http://ros.org/wiki/xacro">
+  <xacro:arg name="current_dirpath" default=""/>
   <xacro:property name="entity_name" value="ground_station_antenna_1"/>
-  <xacro:property name="pos_2d" value="7.5 3"/>
+  <xacro:property name="pos_2d" value="15 3"/>
   <xacro:property name="antenna_height" value="1.8"/>
-  <xacro:include filename="/home/haruki/Desktop/ugv_comms_in_gazebo/models/xacro_base/ground_station_antenna.xacro" />
+  <xacro:include filename="$(arg current_dirpath)/models/xacro_base/ground_station_antenna.xacro" />
   <origin xyz="${pos_2d} ${antenna_height}" rpy="0 0 0"/>
   <xacro:ground_station_antenna name="${entity_name}" antenna_height="${antenna_height}"/>

File: models/ground_station_antennas/xacro/ground_station_antenna_2.xacro (robot description, xacro)
@@ -1,8 +1,9 @@
 <?xml version="1.0"?>
 <robot name="ground_station_antenna_2" xmlns:xacro="http://ros.org/wiki/xacro">
+  <xacro:arg name="current_dirpath" default=""/>
   <xacro:property name="entity_name" value="ground_station_antenna_2"/>
-  <xacro:property name="pos_2d" value="10 3"/>
+  <xacro:property name="pos_2d" value="20 3"/>
   <xacro:property name="antenna_height" value="1.8"/>
-  <xacro:include filename="/home/haruki/Desktop/ugv_comms_in_gazebo/models/xacro_base/ground_station_antenna.xacro" />
+  <xacro:include filename="$(arg current_dirpath)/models/xacro_base/ground_station_antenna.xacro" />
   <origin xyz="${pos_2d} ${antenna_height}" rpy="0 0 0"/>
   <xacro:ground_station_antenna name="${entity_name}" antenna_height="${antenna_height}"/>

File: models/multicopters/xacro/multicopter_0.xacro (robot description, xacro)
@@ -2,7 +2,8 @@
 <robot name="multicopter_0" xmlns:xacro="http://ros.org/wiki/xacro">
   <xacro:property name="entity_name" value="multicopter_0"/>
-  <xacro:include filename="/home/haruki/Desktop/ugv_comms_in_gazebo/models/xacro_base/multicopter.xacro" />
+  <xacro:arg name="current_dirpath" default=""/>
+  <xacro:include filename="$(arg current_dirpath)/models/xacro_base/multicopter.xacro" />
   <!-- <origin xyz="0.0 0.0 0.053302" rpy="0 0 0" /> -->
-  <origin xyz="0.0 0.0 2.0" rpy="0 0 0" />
+  <origin xyz="0 0.0 3.0" rpy="0 0 0" />
   <!-- frame -->
   <xacro:base name="${entity_name}"/>

Commit message: refactering rf_comms_custom

File: models/ground_station_antennas/xacro/ground_station_antenna_0.xacro (robot description, xacro)
@@ -3,5 +3,5 @@
   <xacro:arg name="current_dirpath" default=""/>
   <xacro:property name="entity_name" value="ground_station_antenna_0"/>
-  <xacro:property name="pos_2d" value="10 3"/>
+  <xacro:property name="pos_2d" value="5 3"/>
   <xacro:property name="antenna_height" value="1.8"/>
   <xacro:include filename="$(arg current_dirpath)/models/xacro_base/ground_station_antenna.xacro" />

File: models/ground_station_antennas/xacro/ground_station_antenna_1.xacro (robot description, xacro)
@@ -3,5 +3,5 @@
   <xacro:arg name="current_dirpath" default=""/>
   <xacro:property name="entity_name" value="ground_station_antenna_1"/>
-  <xacro:property name="pos_2d" value="11 3"/>
+  <xacro:property name="pos_2d" value="7 3"/>
   <xacro:property name="antenna_height" value="1.8"/>
   <xacro:include filename="$(arg current_dirpath)/models/xacro_base/ground_station_antenna.xacro" />

File: models/ground_station_antennas/xacro/ground_station_antenna_2.xacro (robot description, xacro)
@@ -3,5 +3,5 @@
   <xacro:arg name="current_dirpath" default=""/>
   <xacro:property name="entity_name" value="ground_station_antenna_2"/>
-  <xacro:property name="pos_2d" value="12 3"/>
+  <xacro:property name="pos_2d" value="9 3"/>
   <xacro:property name="antenna_height" value="1.8"/>
   <xacro:include filename="$(arg current_dirpath)/models/xacro_base/ground_station_antenna.xacro" />

File: models/multicopters/xacro/multicopter_0.xacro (robot description, xacro)
@@ -5,5 +5,5 @@
   <xacro:include filename="$(arg current_dirpath)/models/xacro_base/multicopter.xacro" />
   <!-- <origin xyz="0.0 0.0 0.053302" rpy="0 0 0" /> -->
-  <origin xyz="0 0.0 3.0" rpy="0 0 0" />
+  <origin xyz="0 0.0 2.5" rpy="0 0 0" />
   <!-- frame -->
   <xacro:base name="${entity_name}"/>
