Commit message: fixed and calculate sum of association ]time

File: models/ground_station_antennas/xacro/ground_station_antenna_1.xacro (robot description, xacro)
@@ -3,5 +3,5 @@
   <xacro:arg name="current_dirpath" default=""/>
   <xacro:property name="entity_name" value="ground_station_antenna_1"/>
-  <xacro:property name="pos_2d" value="15 3"/>
+  <xacro:property name="pos_2d" value="11 3"/>
   <xacro:property name="antenna_height" value="1.8"/>
   <xacro:include filename="$(arg current_dirpath)/models/xacro_base/ground_station_antenna.xacro" />

File: models/ground_station_antennas/xacro/ground_station_antenna_2.xacro (robot description, xacro)
@@ -3,5 +3,5 @@
   <xacro:arg name="current_dirpath" default=""/>
   <xacro:property name="entity_name" value="ground_station_antenna_2"/>
-  <xacro:property name="pos_2d" value="20 3"/>
+  <xacro:property name="pos_2d" value="12 3"/>
   <xacro:property name="antenna_height" value="1.8"/>
   <xacro:include filename="$(arg current_dirpath)/models/xacro_base/ground_station_antenna.xacro" />

Commit message: this version results are used in zemi 2024/05/14

File: models/ground_station_antennas/xacro/ground_station_antenna_1.xacro (robot description, xacro)
@@ -3,5 +3,5 @@
   <xacro:arg name="current_dirpath" default=""/>
   <xacro:property name="entity_name" value="ground_station_antenna_1"/>
-  <xacro:property name="pos_2d" value="7 3"/>
+  <xacro:property name="pos_2d" value="5.5 3"/>
   <xacro:property name="antenna_height" value="1.8"/>
   <xacro:include filename="$(arg current_dirpath)/models/xacro_base/ground_station_antenna.xacro" />

File: models/ground_station_antennas/xacro/ground_station_antenna_2.xacro (robot description, xacro)
@@ -3,5 +3,5 @@
   <xacro:arg name="current_dirpath" default=""/>
   <xacro:property name="entity_name" value="ground_station_antenna_2"/>
-  <xacro:property name="pos_2d" value="9 3"/>
+  <xacro:property name="pos_2d" value="6.0 3"/>
   <xacro:property name="antenna_height" value="1.8"/>
   <xacro:include filename="$(arg current_dirpath)/models/xacro_base/ground_station_antenna.xacro" />

File: models/multicopters/xacro/multicopter_0.xacro (robot description, xacro)
@@ -5,5 +5,5 @@
   <xacro:include filename="$(arg current_dirpath)/models/xacro_base/multicopter.xacro" />
   <!-- <origin xyz="0.0 0.0 0.053302" rpy="0 0 0" /> -->
-  <origin xyz="0 0.0 2.5" rpy="0 0 0" />
+  <origin xyz="0.0 0.0 2.0" rpy="0 0 0" />
   <!-- frame -->
   <xacro:base name="${entity_name}"/>
